File: PCB/echoIR.kicad_sch (KiCad schematic)
At the start: 20 parts, among them J1 USB_C_Receptacle_PowerOnly_6P, Q1 AO3400A, SW1 SW_Push

Commit message: Add firmware
Connections:
- net GP16 renamed TSOPOUT
Other:
- moved on the sheet: C3, C4
Changed lines of the file:
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@@
+	)
+	(junction
+		(at 77.47 135.89)
+		(diameter 0)
+		(color 0 0 0 0)
 	)
 	(junction
@@
 	)
 	(junction
-		(at 74.93 135.89)
-		(diameter 0)
-		(color 0 0 0 0)
-	)
-	(junction
 		(at 45.72 92.71)
 		(diameter 0)
@@
 	)
 	(junction
-		(at 74.93 143.51)
-		(diameter 0)
-		(color 0 0 0 0)
-	)
-	(junction
 		(at 57.15 134.62)
 		(diameter 0)
@@
 	)
 	(junction
+		(at 77.47 143.51)
+		(diameter 0)
+		(color 0 0 0 0)
+	)
+	(junction
 		(at 82.55 64.77)
 		(diameter 0)
@@
 	(wire
 		(pts
-			(xy 74.93 135.89) (xy 80.01 135.89)
-		)
-		(stroke
-			(width 0)
-			(type default)
-		)
-	)
-	(wire
-		(pts
 			(xy 55.88 134.62) (xy 57.15 134.62)
 		)
@@
 	(wire
 		(pts
+			(xy 77.47 135.89) (xy 82.55 135.89)
+		)
+		(stroke
+			(width 0)
+			(type default)
+		)
+	)
+	(wire
+		(pts
 			(xy 232.41 102.87) (xy 229.87 102.87)
 		)
@@
 	(wire
 		(pts
+			(xy 77.47 143.51) (xy 82.55 143.51)
+		)
+		(stroke
+			(width 0)
+			(type default)
+		)
+	)
+	(wire
+		(pts
 			(xy 82.55 63.5) (xy 82.55 64.77)
 		)
@@
 	(wire
 		(pts
-			(xy 58.42 143.51) (xy 74.93 143.51)
+			(xy 58.42 143.51) (xy 77.47 143.51)
 		)
 		(stroke
@@
 	(wire
 		(pts
-			(xy 74.93 143.51) (xy 80.01 143.51)
-		)
-		(stroke
-			(width 0)
-			(type default)
-		)
-	)
-	(wire
-		(pts
 			(xy 58.42 144.78) (xy 55.88 144.78)
 		)
@@
 	(wire
 		(pts
-			(xy 74.93 135.89) (xy 57.15 135.89)
+			(xy 57.15 135.89) (xy 77.47 135.89)
 		)
 		(stroke
@@
 		)
 	)
-	(global_label "GP16"
+	(global_label "TSOPOUT"
 		(shape input)
 		(at 55.88 139.7 0)
@@
 		)
 		(property "Intersheetrefs" "${INTERSHEET_REFS}"
-			(at 63.8242 139.7 0)
+			(at 67.2714 139.7 0)
 			(effects
 				(font
@@
 		)
 	)
-	(global_label "GP16"
+	(global_label "TSOPOUT"
 		(shape input)
 		(at 180.34 93.98 0)
@@
 		)
 		(property "Intersheetrefs" "${INTERSHEET_REFS}"
-			(at 188.2842 93.98 0)
+			(at 191.7314 93.98 0)
 			(effects
 				(font
@@
 	(symbol
 		(lib_id "Device:C")
-		(at 80.01 139.7 0)
+		(at 82.55 139.7 0)
 		(unit 1)
 		(exclude_from_sim no)
@@
 		(fields_autoplaced yes)
 		(property "Reference" "C4"
-			(at 83.82 138.4299 0)
+			(at 86.36 138.4299 0)
 			(effects
 				(font
@@
 		)
 		(property "Value" "4.7µF"
-			(at 83.82 140.9699 0)
+			(at 86.36 140.9699 0)
 			(effects
 				(font
@@
 		)
 		(property "Footprint" "Capacitor_SMD:C_1206_3216Metric_Pad1.33x1.80mm_HandSolder"
-			(at 80.9752 143.51 0)
+			(at 83.5152 143.51 0)
 			(effects
 				(font
@@
 		)
 		(property "Datasheet" "~"
-			(at 80.01 139.7 0)
+			(at 82.55 139.7 0)
 			(effects
 				(font
@@
 		)
 		(property "Description" "Unpolarized capacitor"
-			(at 80.01 139.7 0)
+			(at 82.55 139.7 0)
 			(effects
 				(font
@@
 	(symbol
 		(lib_id "Device:C")
-		(at 74.93 139.7 0)
+		(at 77.47 139.7 0)
 		(mirror y)
 		(unit 1)
@@
 		(dnp no)
 		(property "Reference" "C3"
-			(at 71.12 138.4299 0)
+			(at 73.66 138.4299 0)
 			(effects
 				(font
@@
 		)
 		(property "Value" "100nF"
-			(at 71.12 140.9699 0)
+			(at 73.66 140.9699 0)
 			(effects
 				(font
@@
 		)
 		(property "Footprint" "Capacitor_SMD:C_1206_3216Metric_Pad1.33x1.80mm_HandSolder"
-			(at 73.9648 143.51 0)
+			(at 76.5048 143.51 0)
 			(effects
 				(font
@@
 		)
 		(property "Datasheet" "~"
-			(at 74.93 139.7 0)
+			(at 77.47 139.7 0)
 			(effects
 				(font
@@
 		)
 		(property "Description" "Unpolarized capacitor"
-			(at 74.93 139.7 0)
-			(effects
-				(font
+			(at 77.47 139.7 0)
+			(effects
+				(font
